File: ATM90E3x_fw.kicad_pcb (KiCad board)
At the start: 2 copper layers, 50.8 x 50.8 mm, 67 parts, among them IC1 ATM90E36_ATM90E36, J1 RJ45, J2 CONN_01X04, J3 GS3, J4 GS3, J5 GS3, J6 CONN_01X06, J7 CONN_01X06, J8 CONN_01X04, J9 GROVE-SMD-90D, U1 ROF-78E, Y1 Crystal_GND24

Commit message: Arrange parts
Parts:
- R3, R5: moved to B.Cu
- moved R23 77.0 mm to (85.1, 102.9)
- moved R11 73.5 mm to (83.8, 85.1), turned to 90 degrees
- moved R19 73.0 mm to (82.5, 99.1), turned to 90 degrees
- moved R16 67.6 mm to (83.3, 66.0), turned to 90 degrees
- moved R22 66.3 mm to (85.8, 91.4)
- moved R15 66.1 mm to (86.4, 87.6)
- moved R18 66.0 mm to (82.5, 94.7), turned to 90 degrees
- moved R8 65.3 mm to (85.1, 50.8), turned to 90 degrees
- moved R10 64.7 mm to (83.3, 80.8), turned to 90 degrees
- moved C1 63.6 mm to (87.6, 51.3), turned to 270 degrees
- moved R14 63.4 mm to (85.8, 77.5)
- moved C10 61.4 mm to (87.6, 99.1), turned to 90 degrees
- moved R17 60.4 mm to (82.5, 70.6), turned to 90 degrees
- moved R13 60.1 mm to (86.4, 57.1), turned to 180 degrees
- moved R12 56.3 mm to (86.4, 48.3), turned to 180 degrees
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
Commit message: Updated master layout
Parts:
- added C22: 1u/16V, Capacitors_SMD:C_0603, F.Cu at (155.8, 106.9)
- added C23: 100u/16V, Capacitors_SMD:CP_Elec_5x5.8, F.Cu at (163.8, 108.4)
- added C24: 1u/50V, Capacitors_SMD:C_0603, F.Cu at (175.8, 93.7)
- added C25: 220u/50V, Capacitors_SMD:CP_Elec_8x10, F.Cu at (153.9, 97.7)
- added D5: LED, LEDs:LED_0603, F.Cu at (178.7, 82.5)
- added D6: D_Schottky, Diodes_SMD:D_SOD-123, F.Cu at (172.5, 78.0)
- added D7: D_Schottky, Diodes_SMD:D_SOD-123, F.Cu at (163.7, 78.0)
- added D8: D_Schottky, Diodes_SMD:D_SOD-123, F.Cu at (172.5, 84.3)
- added D9: D_Schottky, Diodes_SMD:D_SOD-123, F.Cu at (163.7, 84.3)
- added J10: GROVE-SMD-90D, ATM90E26_from_eagle:SEEED-CONNECTOR--2016_HW4-SMD-2.0-90D, F.Cu at (166.1, 101.5)
- added JP1: Jumper_NC_Small, Connectors:GS2, F.Cu at (145.4, 98.2)
- added LOGO2: LOGO, Whatnick_logo:Whatnick_logo, F.Cu at (147.5, 108.8)
- added R29: R, Resistors_SMD:R_0603_HandSoldering, F.Cu at (179.2, 77.4)
- J1: value RJ45 -> CONN_01X04; footprint Molex_RJ45:RJ45_8 -> Connectors_JST:JST_SH_SM04B-SRSS-TB_04x1.00mm_Angled
- J2: value CONN_01X04 -> GS3; footprint Connectors_Phoenix:PhoenixContact_MC-G_04x3.81mm_Angled -> Connectors:GS3
- J3: value GS3 -> CONN_01X06; footprint Connectors:GS3 -> Connectors_JST:JST_SHL_SM06B-SHLS-TF_06x1.00mm_Angled
- J4: value GS3 -> CONN_01X04; footprint Connectors:GS3 -> Connectors_Phoenix:PhoenixContact_MC-G_04x3.81mm_Angled
- J5: value GS3 -> RJ45; footprint Connectors:GS3 -> Molex_RJ45:RJ45_8
- J6, J7: value CONN_01X06 -> GS3; footprint Connectors_JST:JST_SHL_SM06B-SHLS-TF_06x1.00mm_Angled -> Connectors:GS3
- J8: value CONN_01X04 -> CONN_01X06; footprint Connectors_JST:JST_SH_SM04B-SRSS-TB_04x1.00mm_Angled -> Connectors_JST:JST_SHL_SM06B-SHLS-TF_06x1.00mm_Angled
- J9: value GROVE-SMD-90D -> GS3; footprint ATM90E26_from_eagle:SEEED-CONNECTOR--2016_HW4-SMD-2.0-90D -> Connectors:GS3
- R27: value R -> SMD-RES-ARRAY; footprint Resistors_SMD:R_0603 -> Resistors_SMD:R_Array_Concave_4x0603
- R7: value SMD-RES-ARRAY -> R; footprint Resistors_SMD:R_Array_Concave_4x0603 -> Resistors_SMD:R_0603
Connections:
- net Net-(MS1-Pad11) renamed SCK
- J1 pad 1: I1P_IN -> CF4
- J1 pad 2: I1N_IN -> CF3
- J1 pad 3: I2P_IN -> CF2
- J1 pad 4: I2N_IN -> CF1
- J2 pad 2: UC -> DMA
- J2 pad 3: UB -> +3V3
- J3 pad 1: GND -> VDD
- J3 pad 2: DMA -> MOSI
- J3 pad 3: +3V3 -> MISO
- J4 pad 2: PM0 -> UC
- J4 pad 3: +3V3 -> UB
- J5 pad 1: GND -> I1P_IN
- J5 pad 2: PM1 -> I1N_IN
- J5 pad 3: +3V3 -> I2P_IN
- J6 pad 1: VDD -> GND
- J6 pad 2: MOSI -> PM0
- J6 pad 3: MISO -> +3V3
- J7 pad 1: DMA -> GND
- J7 pad 3: PM0 -> +3V3
- J8 pad 1: CF4 -> DMA
- J8 pad 2: CF3 -> PM1
- J8 pad 3: CF2 -> PM0
- J8 pad 4: CF1 -> IRQ1
- J9 pad 2: Net-(J9-Pad2) -> CS
- J9 pad 3: +3V3 -> Net-(J9-Pad3)
- MS1 pad 12: Net-(MS1-Pad12) -> MOSI
- MS1 pad 13: Net-(MS1-Pad13) -> MISO
- MS1 pad 17: Net-(J9-Pad2) -> Net-(J10-Pad2)
- MS1 pad 18: Net-(J9-Pad1) -> Net-(J10-Pad1)
- MS1 pad 21: Net-(MS1-Pad21) -> Net-(J9-Pad3)
- MS1 pad 22: Net-(MS1-Pad22) -> Net-(J9-Pad1)
- MS1 pad 26: Net-(MS1-Pad26) -> USB
- R1 pad 1: UA -> GND
- R1 pad 2: V1P -> I1P_IN
- R10 pad 1: GND -> V1P
- R10 pad 2: I3P_IN -> GND
- R11 pad 1: I3N_IN -> UB
- R11 pad 2: GND -> V2P
- R12 pad 1: I1P -> V2P
- R12 pad 2: I1P_IN -> GND
- R13 pad 1: I1N -> GND
- R13 pad 2: I1N_IN -> I2P_IN
- R14 pad 1: I3P -> I2N_IN
- R14 pad 2: I3P_IN -> GND
- R15 pad 1: I3N -> GND
- R15 pad 2: I3N_IN -> IP_IN
- R16 pad 1: GND -> IN_IN
- R16 pad 2: I2P_IN -> GND
- R17 pad 1: I2N_IN -> I2P
- R17 pad 2: GND -> I2P_IN
- R18 pad 1: GND -> I2N
- R18 pad 2: IP_IN -> I2N_IN
- R19 pad 1: IN_IN -> IP
- R19 pad 2: GND -> IP_IN
- R2 pad 1: V1P -> I1N_IN
- R20 pad 1: I2P -> IN
- R20 pad 2: I2P_IN -> IN_IN
- R21 pad 1: I2N -> UC
- R21 pad 2: I2N_IN -> V3P
- R22 pad 1: IP -> V3P
- R22 pad 2: IP_IN -> GND
- R23 pad 1: IN -> Net-(C15-Pad2)
- R23 pad 2: IN_IN -> GND
- R24 pad 1: Net-(C15-Pad2) -> Net-(C20-Pad2)
- R25 pad 1: Net-(C20-Pad2) -> +3V3
- R25 pad 2: GND -> Net-(C19-Pad1)
- R26 pad 1: +3V3 -> Net-(C21-Pad2)
- R26 pad 2: Net-(C19-Pad1) -> GND
- R27 pad 1: Net-(C21-Pad2) -> +3V3
- R27 pad 2: GND -> +3V3
- R28 pad 1: +3V3 -> CF4
- R28 pad 2: +3V3 -> CF3
- R28 pad 3: +3V3 -> CF2
- R28 pad 4: +3V3 -> CF1
- R28 pad 5: MOSI -> Net-(D4-Pad2)
- R28 pad 6: MISO -> Net-(D3-Pad2)
- R28 pad 7: SCLK -> Net-(D2-Pad2)
- R28 pad 8: CS -> Net-(D1-Pad2)
- R3 pad 1: UB -> GND
- R3 pad 2: V2P -> I3P_IN
- R4 pad 1: V2P -> I3N_IN
- R5 pad 1: UC -> I1P
- R5 pad 2: V3P -> I1P_IN
- R6 pad 1: V3P -> I1N
- R6 pad 2: GND -> I1N_IN
- R7 pad 1: CF4 -> I3P
- R7 pad 2: CF3 -> I3P_IN
- R8 pad 1: GND -> I3N
- R8 pad 2: I1P_IN -> I3N_IN
- R9 pad 1: I1N_IN -> UA
- R9 pad 2: GND -> V1P
- U1 pad 2: Net-(U1-Pad2) -> GND
- U1 pad 3: Net-(MS1-Pad26) -> Net-(C22-Pad1)

Commit message: Playing with autoplace
Parts:
- D2, D3, D4, J3, J4, J5, R27: moved to F.Cu
- D7, D8, D9: footprint Diodes_SMD:D_SOD-123 -> Diodes_SMD:D_SMA
- J6, J7, J9, LOGO2, R7: moved to B.Cu
- moved R18 78.6 mm to (146.3, 48.8)
- moved R19 76.5 mm to (137.2, 45.5)
- moved C2 72.2 mm to (156.7, 75.4)
- moved C8 70.8 mm to (157.0, 51.1)
- moved R10 70.0 mm to (153.2, 75.9)
- moved R15 69.6 mm to (143.3, 47.5)
- moved R17 67.7 mm to (149.4, 59.7)
- moved R14 61.9 mm to (140.0, 47.5)
- moved C24 61.7 mm to (117.9, 72.6), turned to 270 degrees
- moved D8 60.4 mm to (112.3, 80.0), turned to 180 degrees
- moved R8 60.4 mm to (145.3, 55.6)
- moved R23 60.4 mm to (133.1, 66.3)
- moved R13 60.3 mm to (146.6, 59.7)
- moved C7 59.7 mm to (148.6, 66.8)
- moved C3 59.5 mm to (148.3, 83.8)
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Connections:
- MS1 pad 2: Net-(MS1-Pad2) -> +3V3
- MS1 pad 4: Net-(MS1-Pad4) -> GND

Commit message: Playing with autoplace
Parts:
- moved C11 47.1 mm to (120.7, 53.6)
- moved C12 43.0 mm to (114.6, 44.7)
- moved C9 41.1 mm to (155.7, 81.0)
- moved C5 41.1 mm to (120.7, 61.2)
- moved C18 40.5 mm to (149.6, 86.9)
- moved C2 38.5 mm to (126.0, 52.3)
- moved C8 35.1 mm to (125.7, 67.1)
- moved R10 35.0 mm to (120.7, 63.0), turned to 0 degrees
- moved C16 32.8 mm to (148.3, 81.8), turned to 90 degrees
- moved R3 25.5 mm to (145.3, 48.8)
- moved R19 23.0 mm to (152.7, 62.5)
- moved C17 22.6 mm to (154.9, 85.3)
- moved R5 22.4 mm to (121.7, 66.5)
- moved R17 20.7 mm to (144.3, 79.8)
- moved C7 19.9 mm to (143.8, 86.1)
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
Commit message: Continuing place
Parts:
- C15, C20, C21, R23, R24, R26: moved to F.Cu
- moved Y1 17.1 mm to (122.2, 65.8), turned to 180 degrees
- moved R23 14.8 mm to (120.7, 63.0)
- moved R26 14.2 mm to (120.7, 55.4)
- moved R24 13.6 mm to (120.7, 59.2), turned to 180 degrees
- moved C20 12.3 mm to (120.7, 57.4)
- moved C21 10.4 mm to (120.7, 53.6)
- moved C15 9.65 mm to (120.7, 61.2), turned to 180 degrees
- moved LOGO1 4.26 mm to (129.3, 58.4)
- moved IC1 2.34 mm to (128.3, 58.2), turned to 270 degrees
- moved C2 1.70 mm to (127.5, 51.6)

Commit message: Place progress
Parts:
- C12, C14, C16, C17, C18, C19, R25: moved to F.Cu
- C13: footprint Capacitors_SMD:C_0603 -> Capacitors_SMD:C_0805; moved to F.Cu
- J2: moved to B.Cu
- moved D3 44.5 mm to (109.7, 43.4)
- moved D2 44.5 mm to (109.7, 45.7)
- moved D4 37.4 mm to (113.3, 43.4)
- moved D1 37.4 mm to (113.3, 45.7)
- moved C9 36.2 mm to (139.7, 48.5), turned to 180 degrees
- moved C17 35.7 mm to (124.5, 66.8), turned to 180 degrees
- moved R27 32.6 mm to (146.6, 44.2), turned to 180 degrees
- moved J2 30.0 mm to (127.0, 44.7), turned to 0 degrees
- moved C18 28.1 mm to (137.7, 61.5), turned to 270 degrees
- moved C3 28.0 mm to (135.9, 55.6)
- moved R28 27.3 mm to (120.1, 50.3), turned to 180 degrees
- moved C7 25.1 mm to (135.9, 62.2)
- moved C16 24.5 mm to (128.8, 67.1), turned to 0 degrees
- moved C14 24.0 mm to (133.1, 50.5)
- moved C13 23.0 mm to (132.8, 48.8)
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Connections:
- C11 pad 1: V3P -> V1P
- C5 pad 1: V1P -> V3P
- J3 pad 1: VDD -> +3V3
- R10 pad 1: V1P -> V3P
- R21 pad 2: V3P -> V1P
- R22 pad 1: V3P -> V1P
- R9 pad 2: V1P -> V3P

Commit message: Place completed
Parts:
- added J11: CONN_01X03, Connectors_JST:JST_SH_BM03B-SRSS-TB_03x1.00mm_Straight, F.Cu at (129.0, 43.7)
- C18: footprint Capacitors_SMD:C_0603 -> Capacitors_SMD:C_0805
- J1: footprint Connectors_JST:JST_SH_SM04B-SRSS-TB_04x1.00mm_Angled -> Connectors_JST:JST_SH_BM04B-SRSS-TB_04x1.00mm_Straight
- J3, J8: footprint Connectors_JST:JST_SHL_SM06B-SHLS-TF_06x1.00mm_Angled -> Connectors_JST:JST_SH_BM06B-SRSS-TB_06x1.00mm_Straight
- J4: footprint Connectors_Phoenix:PhoenixContact_MC-G_04x3.81mm_Angled -> Connectors_Phoenix:PhoenixContact_MC-G_04x3.50mm_Angled
- moved C19 25.7 mm to (130.6, 66.5), turned to 270 degrees
- moved J1 23.2 mm to (111.0, 65.8)
- moved J8 22.7 mm to (120.3, 65.8)
- moved D3 17.0 mm to (110.0, 60.5)
- moved D4 17.0 mm to (113.5, 60.5)
- moved D2 16.5 mm to (110.0, 62.2)
- moved D1 16.4 mm to (113.5, 62.1)
- moved C21 11.6 mm to (118.7, 50.7)
- moved R26 11.5 mm to (120.5, 50.8)
- moved R24 11.0 mm to (120.5, 47.5)
- moved R28 10.9 mm to (119.6, 61.2), turned to 270 degrees
- moved C20 10.9 mm to (118.7, 47.5)
- moved R27 10.9 mm to (136.9, 49.3)
- moved C17 10.8 mm to (135.1, 65.0), turned to 0 degrees
- moved C15 10.6 mm to (118.7, 44.1)
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Connections:
- net Net-(C22-Pad1) renamed /Featherwing/VOUT
- net Net-(C24-Pad1) renamed /Featherwing/VIN
Other:
- net class Power: clearance 0.3 -> 0.2; trace_width 0.5 -> 0.4

Commit message: Fixed global names after ERC
Connections:
- net +3V3 renamed VDD
- MS1 pad 11: SCK -> SCLK
