File: ATM90E3x.sch (KiCad schematic (older format))
At the start: 64 parts, among them IC1 ATM90E36_ATM90E36, J1 RJ45, J2 CONN_01X04, J3 GS3, J4 GS3, J5 GS3, J6 CONN_01X06, J7 CONN_01X06, J8 CONN_01X04, Y1 Crystal_GND24

Commit message: Updated master layout
Parts:
- renumbered J8 to J1, J3 to J2, J6 to J3, J2 to J4, J1 to J5, J4 to J6, J5 to J7, J7 to J8, R8 to R1, R2 to R10, R3 to R11, R4 to R12, R16 to R13, R17 to R14, R18 to R15, R19 to R16, R20 to R17, R21 to R18, R22 to R19, R9 to R2, R23 to R20, R5 to R21, R6 to R22, R24 to R23, R25 to R24, R26 to R25, R27 to R26, R28 to R27, R7 to R28, R10 to R3, R11 to R4, R12 to R5, R13 to R6, R14 to R7, R15 to R8, R1 to R9
Changed lines of the file:
@@
 LIBS:ROF-78E
 LIBS:ATM90E26_Featherwing
-LIBS:logo
+LIBS:whatnick
 LIBS:ATM90E3x_fw-cache
 EELAYER 26 0
@@
 $EndComp
 $Comp
-L RJ45 J1
+L RJ45 J5
 U 1 1 5943DD9C
 P 9900 1450
-F 0 "J1" H 9976 2067 50  0000 C CNN
+F 0 "J5" H 9976 2067 50  0000 C CNN
 F 1 "RJ45" H 9976 1976 50  0000 C CNN
 F 2 "Molex_RJ45:RJ45_8" H 9900 1450 50  0001 C CNN
@@
 $EndComp
 $Comp
-L CONN_01X04 J2
+L CONN_01X04 J4
 U 1 1 5943DF45
 P 9800 3500
-F 0 "J2" V 9672 3728 50  0000 L CNN
+F 0 "J4" V 9672 3728 50  0000 L CNN
 F 1 "CONN_01X04" V 9763 3728 50  0000 L CNN
 F 2 "Connectors_Phoenix:PhoenixContact_MC-G_04x3.81mm_Angled" H 9800 3500 50  0001 C CNN
@@
 $EndComp
 $Comp
-L GS3 J3
+L GS3 J2
 U 1 1 59440387
 P 9150 5550
-F 0 "J3" H 9150 5225 50  0000 C CNN
+F 0 "J2" H 9150 5225 50  0000 C CNN
 F 1 "GS3" H 9150 5316 50  0000 C CNN
 F 2 "Connectors:GS3" V 9238 5476 50  0001 C CNN
@@
 $EndComp
 $Comp
-L GS3 J4
+L GS3 J6
 U 1 1 59440489
 P 9900 5550
-F 0 "J4" H 9900 5225 50  0000 C CNN
+F 0 "J6" H 9900 5225 50  0000 C CNN
 F 1 "GS3" H 9900 5316 50  0000 C CNN
 F 2 "Connectors:GS3" V 9988 5476 50  0001 C CNN
@@
 $EndComp
 $Comp
-L GS3 J5
+L GS3 J7
 U 1 1 594404BF
 P 10550 5550
-F 0 "J5" H 10550 5225 50  0000 C CNN
+F 0 "J7" H 10550 5225 50  0000 C CNN
 F 1 "GS3" H 10550 5316 50  0000 C CNN
 F 2 "Connectors:GS3" V 10638 5476 50  0001 C CNN
@@
 $EndComp
 $Comp
-L SEEED-RESISTOR-2016_SMD-RES-ARRAY-1K-4R_RA1206-8_ R7
+L SEEED-RESISTOR-2016_SMD-RES-ARRAY-1K-4R_RA1206-8_ R28
 U 1 1 594405BB
 P 9700 6200
-F 0 "R7" H 9700 6554 45  0000 C CNN
+F 0 "R28" H 9700 6554 45  0000 C CNN
 F 1 "SMD-RES-ARRAY" H 9700 6470 45  0000 C CNN
 F 2 "Resistors_SMD:R_Array_Concave_4x0603" H 9700 6200 60  0001 C CNN
@@
 $EndComp
 $Comp
-L CONN_01X06 J6
+L CONN_01X06 J3
 U 1 1 59440A00
 P 9600 4500
-F 0 "J6" H 9678 4541 50  0000 L CNN
+F 0 "J3" H 9678 4541 50  0000 L CNN
 F 1 "CONN_01X06" H 9678 4450 50  0000 L CNN
 F 2 "Connectors_JST:JST_SHL_SM06B-SHLS-TF_06x1.00mm_Angled" H 9600 4500 50  0001 C CNN
@@
 $EndComp
 $Comp
-L CONN_01X06 J7
+L CONN_01X06 J8
 U 1 1 59440AD4
 P 10700 4500
-F 0 "J7" H 10778 4541 50  0000 L CNN
+F 0 "J8" H 10778 4541 50  0000 L CNN
 F 1 "CONN_01X06" H 10778 4450 50  0000 L CNN
 F 2 "Connectors_JST:JST_SHL_SM06B-SHLS-TF_06x1.00mm_Angled" H 10700 4500 50  0001 C CNN
@@
 $EndComp
 $Comp
-L R R2
+L R R10
 U 1 1 59441213
 P 1200 2850
-F 0 "R2" H 1270 2896 50  0000 L CNN
+F 0 "R10" H 1270 2896 50  0000 L CNN
 F 1 "R" H 1270 2805 50  0000 L CNN
 F 2 "Resistors_SMD:R_0603" V 1130 2850 50  0001 C CNN
@@
 $EndComp
 $Comp
-L R R1
+L R R9
 U 1 1 59441271
 P 1200 2250
-F 0 "R1" H 1270 2296 50  0000 L CNN
+F 0 "R9" H 1270 2296 50  0000 L CNN
 F 1 "R" H 1270 2205 50  0000 L CNN
 F 2 "Resistors_SMD:R_0603" V 1130 2250 50  0001 C CNN
@@
 $EndComp
 $Comp
-L R R3
+L R R11
 U 1 1 594412B3
 P 1850 2250
-F 0 "R3" H 1920 2296 50  0000 L CNN
+F 0 "R11" H 1920 2296 50  0000 L CNN
 F 1 "R" H 1920 2205 50  0000 L CNN
 F 2 "Resistors_SMD:R_0603" V 1780 2250 50  0001 C CNN
@@
 $EndComp
 $Comp
-L R R4
+L R R12
 U 1 1 594412F5
 P 1850 2850
-F 0 "R4" H 1920 2896 50  0000 L CNN
+F 0 "R12" H 1920 2896 50  0000 L CNN
 F 1 "R" H 1920 2805 50  0000 L CNN
 F 2 "Resistors_SMD:R_0603" V 1780 2850 50  0001 C CNN
@@
 $EndComp
 $Comp
-L R R6
+L R R22
 U 1 1 5944133F
 P 2400 2850
-F 0 "R6" H 2470 2896 50  0000 L CNN
+F 0 "R22" H 2470 2896 50  0000 L CNN
 F 1 "R" H 2470 2805 50  0000 L CNN
 F 2 "Resistors_SMD:R_0603" V 2330 2850 50  0001 C CNN
@@
 $EndComp
 $Comp
-L R R5
+L R R21
 U 1 1 59441389
 P 2400 2250
-F 0 "R5" H 2470 2296 50  0000 L CNN
+F 0 "R21" H 2470 2296 50  0000 L CNN
 F 1 "R" H 2470 2205 50  0000 L CNN
 F 2 "Resistors_SMD:R_0603" V 2330 2250 50  0001 C CNN
@@
 $EndComp
 $Comp
-L R R12
+L R R5
 U 1 1 594506E9
 P 1100 4650
-F 0 "R12" V 893 4650 50  0000 C CNN
+F 0 "R5" V 893 4650 50  0000 C CNN
 F 1 "R" V 984 4650 50  0000 C CNN
 F 2 "Resistors_SMD:R_0603" V 1030 4650 50  0001 C CNN
@@
 $EndComp
 $Comp
-L R R13
+L R R6
 U 1 1 594507D2
 P 1100 5450
-F 0 "R13" V 893 5450 50  0000 C CNN
+F 0 "R6" V 893 5450 50  0000 C CNN
 F 1 "R" V 984 5450 50  0000 C CNN
 F 2 "Resistors_SMD:R_0603" V 1030 5450 50  0001 C CNN
@@
 $EndComp
 $Comp
-L R R14
+L R R7
 U 1 1 59450838
 P 1100 5950
-F 0 "R14" V 893 5950 50  0000 C CNN
+F 0 "R7" V 893 5950 50  0000 C CNN
 F 1 "R" V 984 5950 50  0000 C CNN
 F 2 "Resistors_SMD:R_0603" V 1030 5950 50  0001 C CNN
@@
 $EndComp
 $Comp
-L R R15
+L R R8
 U 1 1 5945088A
 P 1100 6700
-F 0 "R15" V 893 6700 50  0000 C CNN
+F 0 "R8" V 893 6700 50  0000 C CNN
 F 1 "R" V 984 6700 50  0000 C CNN
 F 2 "Resistors_SMD:R_0603" V 1030 6700 50  0001 C CNN
@@
 $EndComp
 $Comp
-L R R20
+L R R17
 U 1 1 5945103A
 P 2200 4650
-F 0 "R20" V 1993 4650 50  0000 C CNN
+F 0 "R17" V 1993 4650 50  0000 C CNN
 F 1 "R" V 2084 4650 50  0000 C CNN
 F 2 "Resistors_SMD:R_0603" V 2130 4650 50  0001 C CNN
@@
 $EndComp
 $Comp
-L R R21
+L R R18
 U 1 1 594510B2
 P 2200 5450
-F 0 "R21" V 1993 5450 50  0000 C CNN
+F 0 "R18" V 1993 5450 50  0000 C CNN
 F 1 "R" V 2084 5450 50  0000 C CNN
 F 2 "Resistors_SMD:R_0603" V 2130 5450 50  0001 C CNN
@@
 $EndComp
 $Comp
-L R R22
+L R R19
 U 1 1 59451138
 P 2200 5950
-F 0 "R22" V 1993 5950 50  0000 C CNN
+F 0 "R19" V 1993 5950 50  0000 C CNN
 F 1 "R" V 2084 5950 50  0000 C CNN
 F 2 "Resistors_SMD:R_0603" V 2130 5950 50  0001 C CNN
@@
 $EndComp
 $Comp
-L R R23
+L R R20
 U 1 1 594511B0
 P 2200 6700
-F 0 "R23" V 1993 6700 50  0000 C CNN
+F 0 "R20" V 1993 6700 50  0000 C CNN
 F 1 "R" V 2084 6700 50  0000 C CNN
 F 2 "Resistors_SMD:R_0603" V 2130 6700 50  0001 C CNN
@@
 $EndComp
 $Comp
-L R R8
+L R R1
 U 1 1 594518B6
 P 950 4900
-F 0 "R8" H 880 4854 50  0000 R CNN
+F 0 "R1" H 880 4854 50  0000 R CNN
 F 1 "R" H 880 4945 50  0000 R CNN
 F 2 "Resistors_SMD:R_0603" V 880 4900 50  0001 C CNN
@@
 $EndComp
 $Comp
-L R R9
+L R R2
 U 1 1 59451937
 P 950 5250
-F 0 "R9" H 880 5204 50  0000 R CNN
+F 0 "R2" H 880 5204 50  0000 R CNN
 F 1 "R" H 880 5295 50  0000 R CNN
 F 2 "Resistors_SMD:R_0603" V 880 5250 50  0001 C CNN
@@
 $EndComp
 $Comp
-L R R10
+L R R3
 U 1 1 5945199D
 P 950 6150
-F 0 "R10" H 880 6104 50  0000 R CNN
+F 0 "R3" H 880 6104 50  0000 R CNN
 F 1 "R" H 880 6195 50  0000 R CNN
 F 2 "Resistors_SMD:R_0603" V 880 6150 50  0001 C CNN
@@
 $EndComp
 $Comp
-L R R11
+L R R4
 U 1 1 59451A13
 P 950 6500
-F 0 "R11" H 880 6454 50  0000 R CNN
+F 0 "R4" H 880 6454 50  0000 R CNN
 F 1 "R" H 880 6545 50  0000 R CNN
 F 2 "Resistors_SMD:R_0603" V 880 6500 50  0001 C CNN
@@
 $EndComp
 $Comp
-L R R16
+L R R13
 U 1 1 59451A73
 P 2050 4850
-F 0 "R16" H 1980 4804 50  0000 R CNN
+F 0 "R13" H 1980 4804 50  0000 R CNN
 F 1 "R" H 1980 4895 50  0000 R CNN
 F 2 "Resistors_SMD:R_0603" V 1980 4850 50  0001 C CNN
@@
 $EndComp
 $Comp
-L R R17
+L R R14
 U 1 1 59451AE7
 P 2050 5200
-F 0 "R17" H 1980 5154 50  0000 R CNN
+F 0 "R14" H 1980 5154 50  0000 R CNN
 F 1 "R" H 1980 5245 50  0000 R CNN
 F 2 "Resistors_SMD:R_0603" V 1980 5200 50  0001 C CNN
@@
 $EndComp
 $Comp
-L R R18
+L R R15
 U 1 1 59451B4B
 P 2050 6150
-F 0 "R18" H 1980 6104 50  0000 R CNN
+F 0 "R15" H 1980 6104 50  0000 R CNN
 F 1 "R" H 1980 6195 50  0000 R CNN
 F 2 "Resistors_SMD:R_0603" V 1980 6150 50  0001 C CNN
@@
 $EndComp
 $Comp
-L R R19
+L R R16
 U 1 1 59451BCB
 P 2050 6500
-F 0 "R19" H 1980 6454 50  0000 R CNN
+F 0 "R16" H 1980 6454 50  0000 R CNN
 F 1 "R" H 1980 6545 50  0000 R CNN
 F 2 "Resistors_SMD:R_0603" V 1980 6500 50  0001 C CNN
@@
 Optional Neutral CT
 $Comp
-L SEEED-RESISTOR-2016_SMD-RES-ARRAY-1K-4R_RA1206-8_ R28
+L SEEED-RESISTOR-2016_SMD-RES-ARRAY-1K-4R_RA1206-8_ R27
 U 1 1 59456219
 P 7100 1300
-F 0 "R28" V 7058 1528 45  0000 L CNN
+F 0 "R27" V 7058 1528 45  0000 L CNN
 F 1 "SMD-RES-ARRAY" V 7142 1528 45  0000 L CNN
 F 2 "Resistors_SMD:R_Array_Concave_4x0603" H 7100 1300 60  0001 C CNN
@@
 $EndComp
 $Comp
-L R R24
+L R R23
 U 1 1 59456D76
 P 4650 4850
-F 0 "R24" H 4720 4896 50  0000 L CNN
+F 0 "R23" H 4720 4896 50  0000 L CNN
 F 1 "R" H 4720 4805 50  0000 L CNN
 F 2 "Resistors_SMD:R_0603" V 4580 4850 50  0001 C CNN
@@
 $EndComp
 $Comp
-L R R25
+L R R24
 U 1 1 59456E76
 P 5300 4850
-F 0 "R25" H 5370 4896 50  0000 L CNN
+F 0 "R24" H 5370 4896 50  0000 L CNN
 F 1 "R" H 5370 4805 50  0000 L CNN
 F 2 "Resistors_SMD:R_0603" V 5230 4850 50  0001 C CNN
@@
 $EndComp
 $Comp
-L R R27
+L R R26
 U 1 1 59456F16
 P 5850 4850
-F 0 "R27" H 5920 4896 50  0000 L CNN
+F 0 "R26" H 5920 4896 50  0000 L CNN
 F 1 "R" H 5920 4805 50  0000 L CNN
 F 2 "Resistors_SMD:R_0603" V 5780 4850 50  0001 C CNN
@@
 $EndComp
 $Comp
-L R R26
+L R R25
 U 1 1 59456FB8
 P 5850 950
-F 0 "R26" V 5643 950 50  0000 C CNN
+F 0 "R25" V 5643 950 50  0000 C CNN
 F 1 "R" V 5734 950 50  0000 C CNN
 F 2 "Resistors_SMD:R_0603" V 5780 950 50  0001 C CNN
@@
 $EndComp
 $Comp
-L CONN_01X04 J8
+L CONN_01X04 J1
 U 1 1 594576D4
 P 7500 3450
-F 0 "J8" H 7578 3491 50  0000 L CNN
+F 0 "J1" H 7578 3491 50  0000 L CNN
 F 1 "CONN_01X04" H 7578 3400 50  0000 L CNN
 F 2 "Connectors_JST:JST_SH_SM04B-SRSS-TB_04x1.00mm_Angled" H 7500 3450 50  0001 C CNN

Commit message: Place progress
Parts:
- C13: footprint Capacitors_SMD:C_0603 -> Capacitors_SMD:C_0805
Connections:
- net VDD is gone; now on net +3V3: J3.1 (P1)
- net V1P: now also C11.1, R21.2, R22.1; no longer C5.1, R10.1, R9.2
- net V3P: now also C5.1, R10.1, R9.2; no longer C11.1, R21.2, R22.1
Changed lines of the file:
@@
 F 0 "C13" H 4258 3704 50  0000 R CNN
 F 1 "C_Small" H 4258 3795 50  0000 R CNN
-F 2 "Capacitors_SMD:C_0603" H 4350 3750 50  0001 C CNN
+F 2 "Capacitors_SMD:C_0805" H 4350 3750 50  0001 C CNN
 F 3 "" H 4350 3750 50  0001 C CNN
 	1    4350 3750
@@
 V3P
 Text GLabel 1450 2500 2    60   Input ~ 0
-V1P
+V3P
 Text GLabel 2100 2500 2    60   Input ~ 0
 V2P
 Text GLabel 2650 2500 2    60   Input ~ 0
-V3P
+V1P
+$Comp
+L +3V3 #PWR017
+U 1 1 597C7279
+P 9300 4100
+F 0 "#PWR017" H 9300 3950 50  0001 C CNN
+F 1 "+3V3" H 9315 4273 50  0000 C CNN
+F 2 "" H 9300 4100 50  0001 C CNN
+F 3 "" H 9300 4100 50  0001 C CNN
+	1    9300 4100
+	1    0    0    -1
+$EndComp
+Wire Wire Line
+	9300 4100 9300 4250
+Connection ~ 9300 4250
 $EndSCHEMATC

Commit message: Place completed
Parts:
- added J11: CONN_01X03, Connectors_JST:JST_SH_BM03B-SRSS-TB_03x1.00mm_Straight, symbol CONN_01X03
- C18: footprint Capacitors_SMD:C_0603 -> Capacitors_SMD:C_0805
- J1: footprint Connectors_JST:JST_SH_SM04B-SRSS-TB_04x1.00mm_Angled -> Connectors_JST:JST_SH_BM04B-SRSS-TB_04x1.00mm_Straight
- J3, J8: footprint Connectors_JST:JST_SHL_SM06B-SHLS-TF_06x1.00mm_Angled -> Connectors_JST:JST_SH_BM06B-SRSS-TB_06x1.00mm_Straight
- J4: footprint Connectors_Phoenix:PhoenixContact_MC-G_04x3.81mm_Angled -> Connectors_Phoenix:PhoenixContact_MC-G_04x3.50mm_Angled; manf# (none) -> 20020110-C041A01LF
Connections:
- net ZX0: now also J11.3 (P3)
- net ZX1: now also J11.2 (P2)
- net ZX2: now also J11.1 (P1)
Changed lines of the file:
@@
 F 0 "J4" V 9672 3728 50  0000 L CNN
 F 1 "CONN_01X04" V 9763 3728 50  0000 L CNN
-F 2 "Connectors_Phoenix:PhoenixContact_MC-G_04x3.81mm_Angled" H 9800 3500 50  0001 C CNN
+F 2 "Connectors_Phoenix:PhoenixContact_MC-G_04x3.50mm_Angled" H 9800 3500 50  0001 C CNN
 F 3 "" H 9800 3500 50  0001 C CNN
+F 4 "20020110-C041A01LF" H 9800 3500 60  0001 C CNN "manf#"
 	1    9800 3500
 	0    1    1    0
@@
 F 0 "J3" H 9678 4541 50  0000 L CNN
 F 1 "CONN_01X06" H 9678 4450 50  0000 L CNN
-F 2 "Connectors_JST:JST_SHL_SM06B-SHLS-TF_06x1.00mm_Angled" H 9600 4500 50  0001 C CNN
+F 2 "Connectors_JST:JST_SH_BM06B-SRSS-TB_06x1.00mm_Straight" H 9600 4500 50  0001 C CNN
 F 3 "" H 9600 4500 50  0001 C CNN
 	1    9600 4500
@@
 F 0 "J8" H 10778 4541 50  0000 L CNN
 F 1 "CONN_01X06" H 10778 4450 50  0000 L CNN
-F 2 "Connectors_JST:JST_SHL_SM06B-SHLS-TF_06x1.00mm_Angled" H 10700 4500 50  0001 C CNN
+F 2 "Connectors_JST:JST_SH_BM06B-SRSS-TB_06x1.00mm_Straight" H 10700 4500 50  0001 C CNN
 F 3 "" H 10700 4500 50  0001 C CNN
 	1    10700 4500
@@
 F 0 "C18" V 5121 1400 50  0000 C CNN
 F 1 "C_Small" V 5212 1400 50  0000 C CNN
-F 2 "Capacitors_SMD:C_0603" H 5350 1400 50  0001 C CNN
+F 2 "Capacitors_SMD:C_0805" H 5350 1400 50  0001 C CNN
 F 3 "" H 5350 1400 50  0001 C CNN
 	1    5350 1400
@@
 F 0 "J1" H 7578 3491 50  0000 L CNN
 F 1 "CONN_01X04" H 7578 3400 50  0000 L CNN
-F 2 "Connectors_JST:JST_SH_SM04B-SRSS-TB_04x1.00mm_Angled" H 7500 3450 50  0001 C CNN
+F 2 "Connectors_JST:JST_SH_BM04B-SRSS-TB_04x1.00mm_Straight" H 7500 3450 50  0001 C CNN
 F 3 "" H 7500 3450 50  0001 C CNN
 	1    7500 3450
@@
 	6300 4200 7650 4200
 Wire Wire Line
-	6500 4100 7650 4100
+	6500 4100 7800 4100
 Wire Wire Line
 	6400 4100 6400 4150
 Wire Wire Line
-	6400 4150 7650 4150
+	6400 4150 8000 4150
 Wire Wire Line
 	4900 3500 4350 3500
@@
 	9300 4100 9300 4250
 Connection ~ 9300 4250
+$Comp
+L CONN_01X03 J11
+U 1 1 597C8259
+P 8200 4150
+F 0 "J11" H 8278 4191 50  0000 L CNN
+F 1 "CONN_01X03" H 8278 4100 50  0000 L CNN
+F 2 "Connectors_JST:JST_SH_BM03B-SRSS-TB_03x1.00mm_Straight" H 8200 4150 50  0001 C CNN
+F 3 "" H 8200 4150 50  0001 C CNN
+	1    8200 4150
+	1    0    0    -1
+$EndComp
+Wire Wire Line
+	7800 4100 7800 4050
+Wire Wire Line
+	7800 4050 8000 4050
+Wire Wire Line
+	8000 4250 7650 4250
+Wire Wire Line
+	7650 4250 7650 4200
 $EndSCHEMATC
