File: ATM90E3x.sch (KiCad schematic (older format))
At the start: 65 parts, among them IC1 ATM90E36_ATM90E36, J1 CONN_01X04, J11 CONN_01X03, J2 GS3, J3 CONN_01X06, J4 CONN_01X04, J5 Conn_01x08, J6 GS3, J7 GS3, J8 CONN_01X06, Y1 Crystal_GND24

Commit message: Add values for additional parts
Parts:
- C1, C10, C11, C15, C2, C20, C21, C3, C4, C5, C6, C7, C8, C9: value C_Small -> 18nF
- C13: value C_Small -> 10uF
- C14: value C_Small -> 100nF
- R1, R13, R14, R15, R16, R2, R4: value R -> 2.4R
- R10, R12, R17, R18, R19, R20, R22, R23, R24, R26, R5, R6, R7, R8: value R -> 1K
- R11, R21, R9: value R -> 100K
Changed lines of the file:
@@
 P 1200 2850
 F 0 "R10" H 1270 2896 50  0000 L CNN
-F 1 "R" H 1270 2805 50  0000 L CNN
+F 1 "1K" H 1270 2805 50  0000 L CNN
 F 2 "Resistors_SMD:R_0603" V 1130 2850 50  0001 C CNN
 F 3 "" H 1200 2850 50  0001 C CNN
@@
 P 1200 2250
 F 0 "R9" H 1270 2296 50  0000 L CNN
-F 1 "R" H 1270 2205 50  0000 L CNN
+F 1 "100K" H 1270 2205 50  0000 L CNN
 F 2 "Resistors_SMD:R_0603" V 1130 2250 50  0001 C CNN
 F 3 "" H 1200 2250 50  0001 C CNN
@@
 P 1850 2250
 F 0 "R11" H 1920 2296 50  0000 L CNN
-F 1 "R" H 1920 2205 50  0000 L CNN
+F 1 "100K" H 1920 2205 50  0000 L CNN
 F 2 "Resistors_SMD:R_0603" V 1780 2250 50  0001 C CNN
 F 3 "" H 1850 2250 50  0001 C CNN
@@
 P 1850 2850
 F 0 "R12" H 1920 2896 50  0000 L CNN
-F 1 "R" H 1920 2805 50  0000 L CNN
+F 1 "1K" H 1920 2805 50  0000 L CNN
 F 2 "Resistors_SMD:R_0603" V 1780 2850 50  0001 C CNN
 F 3 "" H 1850 2850 50  0001 C CNN
@@
 P 2400 2850
 F 0 "R22" H 2470 2896 50  0000 L CNN
-F 1 "R" H 2470 2805 50  0000 L CNN
+F 1 "1K" H 2470 2805 50  0000 L CNN
 F 2 "Resistors_SMD:R_0603" V 2330 2850 50  0001 C CNN
 F 3 "" H 2400 2850 50  0001 C CNN
@@
 P 2400 2250
 F 0 "R21" H 2470 2296 50  0000 L CNN
-F 1 "R" H 2470 2205 50  0000 L CNN
+F 1 "100K" H 2470 2205 50  0000 L CNN
 F 2 "Resistors_SMD:R_0603" V 2330 2250 50  0001 C CNN
 F 3 "" H 2400 2250 50  0001 C CNN
@@
 P 1450 2850
 F 0 "C5" H 1542 2896 50  0000 L CNN
-F 1 "C_Small" H 1542 2805 50  0000 L CNN
+F 1 "18nF" H 1542 2805 50  0000 L CNN
 F 2 "Capacitors_SMD:C_0603" H 1450 2850 50  0001 C CNN
 F 3 "" H 1450 2850 50  0001 C CNN
@@
 P 2100 2850
 F 0 "C6" H 2192 2896 50  0000 L CNN
-F 1 "C_Small" H 2192 2805 50  0000 L CNN
+F 1 "18nF" H 2192 2805 50  0000 L CNN
 F 2 "Capacitors_SMD:C_0603" H 2100 2850 50  0001 C CNN
 F 3 "" H 2100 2850 50  0001 C CNN
@@
 P 2650 2850
 F 0 "C11" H 2742 2896 50  0000 L CNN
-F 1 "C_Small" H 2742 2805 50  0000 L CNN
+F 1 "18nF" H 2742 2805 50  0000 L CNN
 F 2 "Capacitors_SMD:C_0603" H 2650 2850 50  0001 C CNN
 F 3 "" H 2650 2850 50  0001 C CNN
@@
 P 1100 4650
 F 0 "R5" V 893 4650 50  0000 C CNN
-F 1 "R" V 984 4650 50  0000 C CNN
+F 1 "1K" V 984 4650 50  0000 C CNN
 F 2 "Resistors_SMD:R_0603" V 1030 4650 50  0001 C CNN
 F 3 "" H 1100 4650 50  0001 C CNN
@@
 P 1100 5450
 F 0 "R6" V 893 5450 50  0000 C CNN
-F 1 "R" V 984 5450 50  0000 C CNN
+F 1 "1K" V 984 5450 50  0000 C CNN
 F 2 "Resistors_SMD:R_0603" V 1030 5450 50  0001 C CNN
 F 3 "" H 1100 5450 50  0001 C CNN
@@
 P 1100 5950
 F 0 "R7" V 893 5950 50  0000 C CNN
-F 1 "R" V 984 5950 50  0000 C CNN
+F 1 "1K" V 984 5950 50  0000 C CNN
 F 2 "Resistors_SMD:R_0603" V 1030 5950 50  0001 C CNN
 F 3 "" H 1100 5950 50  0001 C CNN
@@
 P 1100 6700
 F 0 "R8" V 893 6700 50  0000 C CNN
-F 1 "R" V 984 6700 50  0000 C CNN
+F 1 "1K" V 984 6700 50  0000 C CNN
 F 2 "Resistors_SMD:R_0603" V 1030 6700 50  0001 C CNN
 F 3 "" H 1100 6700 50  0001 C CNN
@@
 P 2200 4650
 F 0 "R17" V 1993 4650 50  0000 C CNN
-F 1 "R" V 2084 4650 50  0000 C CNN
+F 1 "1K" V 2084 4650 50  0000 C CNN
 F 2 "Resistors_SMD:R_0603" V 2130 4650 50  0001 C CNN
 F 3 "" H 2200 4650 50  0001 C CNN
@@
 P 2200 5450
 F 0 "R18" V 1993 5450 50  0000 C CNN
-F 1 "R" V 2084 5450 50  0000 C CNN
+F 1 "1K" V 2084 5450 50  0000 C CNN
 F 2 "Resistors_SMD:R_0603" V 2130 5450 50  0001 C CNN
 F 3 "" H 2200 5450 50  0001 C CNN
@@
 P 2200 5950
 F 0 "R19" V 1993 5950 50  0000 C CNN
-F 1 "R" V 2084 5950 50  0000 C CNN
+F 1 "1K" V 2084 5950 50  0000 C CNN
 F 2 "Resistors_SMD:R_0603" V 2130 5950 50  0001 C CNN
 F 3 "" H 2200 5950 50  0001 C CNN
@@
 P 2200 6700
 F 0 "R20" V 1993 6700 50  0000 C CNN
-F 1 "R" V 2084 6700 50  0000 C CNN
+F 1 "1K" V 2084 6700 50  0000 C CNN
 F 2 "Resistors_SMD:R_0603" V 2130 6700 50  0001 C CNN
 F 3 "" H 2200 6700 50  0001 C CNN
@@
 P 950 4900
 F 0 "R1" H 880 4854 50  0000 R CNN
-F 1 "R" H 880 4945 50  0000 R CNN
+F 1 "2.4R" H 880 4945 50  0000 R CNN
 F 2 "Resistors_SMD:R_0603" V 880 4900 50  0001 C CNN
 F 3 "" H 950 4900 50  0001 C CNN
@@
 P 950 5250
 F 0 "R2" H 880 5204 50  0000 R CNN
-F 1 "R" H 880 5295 50  0000 R CNN
+F 1 "2.4R" H 880 5295 50  0000 R CNN
 F 2 "Resistors_SMD:R_0603" V 880 5250 50  0001 C CNN
 F 3 "" H 950 5250 50  0001 C CNN
@@
 P 950 6500
 F 0 "R4" H 880 6454 50  0000 R CNN
-F 1 "R" H 880 6545 50  0000 R CNN
+F 1 "2.4R" H 880 6545 50  0000 R CNN
 F 2 "Resistors_SMD:R_0603" V 880 6500 50  0001 C CNN
 F 3 "" H 950 6500 50  0001 C CNN
@@
 P 2050 4850
 F 0 "R13" H 1980 4804 50  0000 R CNN
-F 1 "R" H 1980 4895 50  0000 R CNN
+F 1 "2.4R" H 1980 4895 50  0000 R CNN
 F 2 "Resistors_SMD:R_0603" V 1980 4850 50  0001 C CNN
 F 3 "" H 2050 4850 50  0001 C CNN
@@
 P 2050 5200
 F 0 "R14" H 1980 5154 50  0000 R CNN
-F 1 "R" H 1980 5245 50  0000 R CNN
+F 1 "2.4R" H 1980 5245 50  0000 R CNN
 F 2 "Resistors_SMD:R_0603" V 1980 5200 50  0001 C CNN
 F 3 "" H 2050 5200 50  0001 C CNN
@@
 P 2050 6150
 F 0 "R15" H 1980 6104 50  0000 R CNN
-F 1 "R" H 1980 6195 50  0000 R CNN
+F 1 "2.4R" H 1980 6195 50  0000 R CNN
 F 2 "Resistors_SMD:R_0603" V 1980 6150 50  0001 C CNN
 F 3 "" H 2050 6150 50  0001 C CNN
@@
 P 2050 6500
 F 0 "R16" H 1980 6454 50  0000 R CNN
-F 1 "R" H 1980 6545 50  0000 R CNN
+F 1 "2.4R" H 1980 6545 50  0000 R CNN
 F 2 "Resistors_SMD:R_0603" V 1980 6500 50  0001 C CNN
 F 3 "" H 2050 6500 50  0001 C CNN
@@
 P 1300 4850
 F 0 "C1" H 1392 4896 50  0000 L CNN
-F 1 "C_Small" H 1392 4805 50  0000 L CNN
+F 1 "18nF" H 1392 4805 50  0000 L CNN
 F 2 "Capacitors_SMD:C_0603" H 1300 4850 50  0001 C CNN
 F 3 "" H 1300 4850 50  0001 C CNN
@@
 P 1300 5200
 F 0 "C2" H 1392 5246 50  0000 L CNN
-F 1 "C_Small" H 1392 5155 50  0000 L CNN
+F 1 "18nF" H 1392 5155 50  0000 L CNN
 F 2 "Capacitors_SMD:C_0603" H 1300 5200 50  0001 C CNN
 F 3 "" H 1300 5200 50  0001 C CNN
@@
 P 1300 6150
 F 0 "C3" H 1392 6196 50  0000 L CNN
-F 1 "C_Small" H 1392 6105 50  0000 L CNN
+F 1 "18nF" H 1392 6105 50  0000 L CNN
 F 2 "Capacitors_SMD:C_0603" H 1300 6150 50  0001 C CNN
 F 3 "" H 1300 6150 50  0001 C CNN
@@
 P 1300 6500
 F 0 "C4" H 1392 6546 50  0000 L CNN
-F 1 "C_Small" H 1392 6455 50  0000 L CNN
+F 1 "18nF" H 1392 6455 50  0000 L CNN
 F 2 "Capacitors_SMD:C_0603" H 1300 6500 50  0001 C CNN
 F 3 "" H 1300 6500 50  0001 C CNN
@@
 P 2400 4850
 F 0 "C7" H 2492 4896 50  0000 L CNN
-F 1 "C_Small" H 2492 4805 50  0000 L CNN
+F 1 "18nF" H 2492 4805 50  0000 L CNN
 F 2 "Capacitors_SMD:C_0603" H 2400 4850 50  0001 C CNN
 F 3 "" H 2400 4850 50  0001 C CNN
@@
 P 2400 5200
 F 0 "C8" H 2492 5246 50  0000 L CNN
-F 1 "C_Small" H 2492 5155 50  0000 L CNN
+F 1 "18nF" H 2492 5155 50  0000 L CNN
 F 2 "Capacitors_SMD:C_0603" H 2400 5200 50  0001 C CNN
 F 3 "" H 2400 5200 50  0001 C CNN
@@
 P 2400 6150
 F 0 "C9" H 2492 6196 50  0000 L CNN
-F 1 "C_Small" H 2492 6105 50  0000 L CNN
+F 1 "18nF" H 2492 6105 50  0000 L CNN
 F 2 "Capacitors_SMD:C_0603" H 2400 6150 50  0001 C CNN
 F 3 "" H 2400 6150 50  0001 C CNN
@@
 P 2400 6500
 F 0 "C10" H 2492 6546 50  0000 L CNN
-F 1 "C_Small" H 2492 6455 50  0000 L CNN
+F 1 "18nF" H 2492 6455 50  0000 L CNN
 F 2 "Capacitors_SMD:C_0603" H 2400 6500 50  0001 C CNN
 F 3 "" H 2400 6500 50  0001 C CNN
@@
 P 4350 3750
 F 0 "C13" H 4258 3704 50  0000 R CNN
-F 1 "C_Small" H 4258 3795 50  0000 R CNN
+F 1 "10uF" H 4258 3795 50  0000 R CNN
 F 2 "Capacitors_SMD:C_0805" H 4350 3750 50  0001 C CNN
 F 3 "" H 4350 3750 50  0001 C CNN
@@
 P 4600 3750
 F 0 "C14" H 4508 3704 50  0000 R CNN
-F 1 "C_Small" H 4508 3795 50  0000 R CNN
+F 1 "100nF" H 4508 3795 50  0000 R CNN
 F 2 "Capacitors_SMD:C_0603" H 4600 3750 50  0001 C CNN
 F 3 "" H 4600 3750 50  0001 C CNN
@@
 P 4850 4850
 F 0 "C15" H 4758 4804 50  0000 R CNN
-F 1 "C_Small" H 4758 4895 50  0000 R CNN
+F 1 "18nF" H 4758 4895 50  0000 R CNN
 F 2 "Capacitors_SMD:C_0603" H 4850 4850 50  0001 C CNN
 F 3 "" H 4850 4850 50  0001 C CNN
@@
 P 5450 4850
 F 0 "C20" H 5358 4804 50  0000 R CNN
-F 1 "C_Small" H 5358 4895 50  0000 R CNN
+F 1 "18nF" H 5358 4895 50  0000 R CNN
 F 2 "Capacitors_SMD:C_0603" H 5450 4850 50  0001 C CNN
 F 3 "" H 5450 4850 50  0001 C CNN
@@
 P 6050 4850
 F 0 "C21" H 5958 4804 50  0000 R CNN
-F 1 "C_Small" H 5958 4895 50  0000 R CNN
+F 1 "18nF" H 5958 4895 50  0000 R CNN
 F 2 "Capacitors_SMD:C_0603" H 6050 4850 50  0001 C CNN
 F 3 "" H 6050 4850 50  0001 C CNN
@@
 P 4650 4850
 F 0 "R23" H 4720 4896 50  0000 L CNN
-F 1 "R" H 4720 4805 50  0000 L CNN
+F 1 "1K" H 4720 4805 50  0000 L CNN
 F 2 "Resistors_SMD:R_0603" V 4580 4850 50  0001 C CNN
 F 3 "" H 4650 4850 50  0001 C CNN
@@
 P 5300 4850
 F 0 "R24" H 5370 4896 50  0000 L CNN
-F 1 "R" H 5370 4805 50  0000 L CNN
+F 1 "1K" H 5370 4805 50  0000 L CNN
 F 2 "Resistors_SMD:R_0603" V 5230 4850 50  0001 C CNN
 F 3 "" H 5300 4850 50  0001 C CNN
@@
 P 5850 4850
 F 0 "R26" H 5920 4896 50  0000 L CNN
-F 1 "R" H 5920 4805 50  0000 L CNN
+F 1 "1K" H 5920 4805 50  0000 L CNN
 F 2 "Resistors_SMD:R_0603" V 5780 4850 50  0001 C CNN
 F 3 "" H 5850 4850 50  0001 C CNN

Commit message: Update parts
Parts:
- C12, C16, C17, C19: value C_Small -> 100nF
- C18: value C_Small -> 10uF
- J11: manf# (none) -> BM03B-SRSS-TB(LF)(SN)
- J2: DNP  (none) -> (none)
- J3, J8: manf# (none) -> BM06B-SRSS-TB(LF)(SN)
- J5: manf# (none) -> 105314-1108
- J6, J7: DNP (none) -> (none)
- R25: value R -> 10K
- R27: value SMD-RES-ARRAY -> 10KX4; manf# (none) -> YC164-JR-07510KL
- R28: value SMD-RES-ARRAY -> 1KX4; manf# (none) -> CAT16-102J4LF
- R3: value R -> 2.4R
- Y1: manf# (none) -> ABM10-16.000MHZ-E20-T
Changed lines of the file:
@@
 F 2 "Connectors:GS3" V 9238 5476 50  0001 C CNN
 F 3 "" H 9150 5550 50  0001 C CNN
+F 4 " " H 9150 5550 50  0001 C CNN "DNP "
 	1    9150 5550
 	-1   0    0    1
@@
 F 2 "Connectors:GS3" V 9988 5476 50  0001 C CNN
 F 3 "" H 9900 5550 50  0001 C CNN
+F 4 " " H 9900 5550 50  0001 C CNN "DNP"
 	1    9900 5550
 	-1   0    0    1
@@
 F 2 "Connectors:GS3" V 10638 5476 50  0001 C CNN
 F 3 "" H 10550 5550 50  0001 C CNN
+F 4 " " H 10550 5550 50  0001 C CNN "DNP"
 	1    10550 5550
 	-1   0    0    1
@@
 P 9700 6200
 F 0 "R28" H 9700 6554 45  0000 C CNN
-F 1 "SMD-RES-ARRAY" H 9700 6470 45  0000 C CNN
+F 1 "1KX4" H 9700 6470 45  0000 C CNN
 F 2 "Resistors_SMD:R_Array_Concave_4x0603" H 9700 6200 60  0001 C CNN
 F 3 "" H 9700 6200 60  0001 C CNN
+F 4 "CAT16-102J4LF" H 9700 6200 50  0001 C CNN "manf#"
 	1    9700 6200
 	1    0    0    -1
@@
 F 2 "Connectors_JST:JST_SH_BM06B-SRSS-TB_06x1.00mm_Straight" H 9600 4500 50  0001 C CNN
 F 3 "" H 9600 4500 50  0001 C CNN
+F 4 "BM06B-SRSS-TB(LF)(SN)" H 9600 4500 50  0001 C CNN "manf#"
 	1    9600 4500
 	1    0    0    -1
@@
 F 2 "Connectors_JST:JST_SH_BM06B-SRSS-TB_06x1.00mm_Straight" H 10700 4500 50  0001 C CNN
 F 3 "" H 10700 4500 50  0001 C CNN
+F 4 "BM06B-SRSS-TB(LF)(SN)" H 10700 4500 50  0001 C CNN "manf#"
 	1    10700 4500
 	1    0    0    -1
@@
 P 950 6150
 F 0 "R3" H 880 6104 50  0000 R CNN
-F 1 "R" H 880 6195 50  0000 R CNN
+F 1 "2.4R" H 880 6195 50  0000 R CNN
 F 2 "Resistors_SMD:R_0603" V 880 6150 50  0001 C CNN
 F 3 "" H 950 6150 50  0001 C CNN
@@
 P 7100 1300
 F 0 "R27" V 7058 1528 45  0000 L CNN
-F 1 "SMD-RES-ARRAY" V 7142 1528 45  0000 L CNN
+F 1 "10KX4" V 7142 1528 45  0000 L CNN
 F 2 "Resistors_SMD:R_Array_Concave_4x0603" H 7100 1300 60  0001 C CNN
 F 3 "" H 7100 1300 60  0001 C CNN
+F 4 "YC164-JR-07510KL" H 7100 1300 50  0001 C CNN "manf#"
 	1    7100 1300
 	0    1    1    0
@@
 P 4350 1900
 F 0 "C12" V 4121 1900 50  0000 C CNN
-F 1 "C_Small" V 4212 1900 50  0000 C CNN
+F 1 "100nF" V 4212 1900 50  0000 C CNN
 F 2 "Capacitors_SMD:C_0603" H 4350 1900 50  0001 C CNN
 F 3 "" H 4350 1900 50  0001 C CNN
@@
 P 5000 1550
 F 0 "C16" V 4771 1550 50  0000 C CNN
-F 1 "C_Small" V 4862 1550 50  0000 C CNN
+F 1 "100nF" V 4862 1550 50  0000 C CNN
 F 2 "Capacitors_SMD:C_0603" H 5000 1550 50  0001 C CNN
 F 3 "" H 5000 1550 50  0001 C CNN
@@
 P 5350 1400
 F 0 "C18" V 5121 1400 50  0000 C CNN
-F 1 "C_Small" V 5212 1400 50  0000 C CNN
+F 1 "10uF" V 5212 1400 50  0000 C CNN
 F 2 "Capacitors_SMD:C_0805" H 5350 1400 50  0001 C CNN
 F 3 "" H 5350 1400 50  0001 C CNN
@@
 P 5350 1200
 F 0 "C17" V 5121 1200 50  0000 C CNN
-F 1 "C_Small" V 5212 1200 50  0000 C CNN
+F 1 "100nF" V 5212 1200 50  0000 C CNN
 F 2 "Capacitors_SMD:C_0603" H 5350 1200 50  0001 C CNN
 F 3 "" H 5350 1200 50  0001 C CNN
@@
 P 5450 950
 F 0 "C19" V 5221 950 50  0000 C CNN
-F 1 "C_Small" V 5312 950 50  0000 C CNN
+F 1 "100nF" V 5312 950 50  0000 C CNN
 F 2 "Capacitors_SMD:C_0603" H 5450 950 50  0001 C CNN
 F 3 "" H 5450 950 50  0001 C CNN
@@
 P 5850 950
 F 0 "R25" V 5643 950 50  0000 C CNN
-F 1 "R" V 5734 950 50  0000 C CNN
+F 1 "10K" V 5734 950 50  0000 C CNN
 F 2 "Resistors_SMD:R_0603" V 5780 950 50  0001 C CNN
 F 3 "" H 5850 950 50  0001 C CNN
@@
 F 2 "Crystals:Crystal_SMD_2520-4pin_2.5x2.0mm" H 6900 4650 50  0001 C CNN
 F 3 "" H 6900 4650 50  0001 C CNN
+F 4 "ABM10-16.000MHZ-E20-T" H 6900 4650 50  0001 C CNN "manf#"
 	1    6900 4650
 	1    0    0    -1
@@
 F 2 "Connectors_JST:JST_SH_BM03B-SRSS-TB_03x1.00mm_Straight" H 8200 4150 50  0001 C CNN
 F 3 "" H 8200 4150 50  0001 C CNN
+F 4 "BM03B-SRSS-TB(LF)(SN)" H 8200 4150 50  0001 C CNN "manf#"
 	1    8200 4150
 	1    0    0    -1
@@
 F 2 "Connector_Molex:Molex_Nano-Fit_105314-xx08_2x04_P2.50mm_Horizontal" H 9850 1700 50  0001 C CNN
 F 3 "~" H 9850 1700 50  0001 C CNN
+F 4 "105314-1108" H 9850 1700 50  0001 C CNN "manf#"
 	1    9850 1700
 	0    -1   -1   0
