File: featherwing.sch (KiCad schematic (older format))
At the start: 16 parts, among them J10 GROVE-SMD-90D, J9 GS3, U1 ROF-78E

Commit message: Add values for additional parts
Parts:
- U1: manf# (none) -> ROF-78E5.0-0.5SMD-R
Changed lines of the file:
@@
 F 2 "ROF-78E:SMD-4" H 2750 3450 50  0001 L CNN
 F 3 "" H 2750 3450 60  0001 C CNN
+F 4 "ROF-78E5.0-0.5SMD-R" H 2750 3450 50  0001 C CNN "manf#"
 	1    2750 3450
 	-1   0    0    -1

Commit message: Update parts
Parts:
- R29: value R -> 1K
Changed lines of the file:
@@
 P 950 3450
 F 0 "R29" V 1030 3450 50  0000 C CNN
-F 1 "R" V 950 3450 50  0000 C CNN
+F 1 "1K" V 950 3450 50  0000 C CNN
 F 2 "Resistors_SMD:R_0603_HandSoldering" V 880 3450 50  0001 C CNN
 F 3 "" H 950 3450 50  0001 C CNN
